Commit message: Update urdf

File: onrobot_rg_description/urdf/onrobot_rg2_model_macro.xacro (robot description, xacro)
@@ -97,4 +97,13 @@
     </gazebo>
   </xacro:macro>
+  <xacro:macro name="pad_contact" params="prefix fingerprefix">
+    <link name="${prefix}${fingerprefix}_pad_contact">
+      <inertial>
+        <origin xyz="0.0 0.0 0.0" rpy="0 0 0" />
+        <mass value="0.0" />
+        <inertia ixx="0.0" ixy="0.0" ixz="0.0" iyy="0.0" iyz="0.0" izz="0.0" />
+      </inertial>
+    </link>
+  </xacro:macro>
   <xacro:macro name="inner_knuckle_joint" params="prefix fingerprefix reflect">
     <joint name="${prefix}${fingerprefix}_inner_knuckle_joint" type="revolute">
@@ -139,4 +148,11 @@
     <xacro:finger_joints prefix="${prefix}" fingerprefix="right" reflect="-1.0"/>
   </xacro:macro>
+  <xacro:macro name="pad_contact_joint" params="prefix fingerprefix">
+    <joint name="${prefix}{fingerprefix}_pad_contact_joint" type="fixed">
+      <origin xyz="0 0.019 0.037" rpy="0 0 0" />
+      <parent link="${prefix}${fingerprefix}_inner_finger" />
+      <child link="${prefix}${fingerprefix}_pad_contact" />
+    </joint>
+  </xacro:macro>
   <xacro:macro name="onrobot_rg2" params="prefix">
     <xacro:onrobot_rg2_base_link prefix="${prefix}"/>
@@ -145,4 +161,8 @@
     <xacro:finger_joint prefix="${prefix}"/>
     <xacro:right_outer_knuckle_joint prefix="${prefix}"/>
+    <xacro:pad_contact prefix="${prefix}" fingerprefix="left"/>
+    <!-- <xacro:pad_contact prefix="${prefix}" fingerprefix="right"/> -->
+    <xacro:pad_contact_joint prefix="${prefix}" fingerprefix="left"/>
+    <!-- <xacro:pad_contact_joint prefix="${prefix}" fingerprefix="right"/> -->
     <xacro:onrobot_rg2_transmission prefix="${prefix}"/>
     <xacro:onrobot_rg2_gazebo prefix="${prefix}"/>

File: onrobot_rg_description/urdf/onrobot_rg6_model_macro.xacro (robot description, xacro)
@@ -96,4 +96,13 @@
     </gazebo>
   </xacro:macro>
+  <xacro:macro name="pad_contact" params="prefix fingerprefix">
+    <link name="${prefix}${fingerprefix}_pad_contact">
+      <inertial>
+        <origin xyz="0.0 0.0 0.0" rpy="0 0 0" />
+        <mass value="0.0" />
+        <inertia ixx="0.0" ixy="0.0" ixz="0.0" iyy="0.0" iyz="0.0" izz="0.0" />
+      </inertial>
+    </link>
+  </xacro:macro>
   <xacro:macro name="inner_knuckle_joint" params="prefix fingerprefix reflect">
     <joint name="${prefix}${fingerprefix}_inner_knuckle_joint" type="revolute">
@@ -138,4 +147,11 @@
     <xacro:finger_joints prefix="${prefix}" fingerprefix="right" reflect="-1.0"/>
   </xacro:macro>
+  <xacro:macro name="pad_contact_joint" params="prefix fingerprefix">
+    <joint name="${prefix}{fingerprefix}_pad_contact_joint" type="fixed">
+      <origin xyz="0 0.0245 0.055" rpy="0 0 0" />
+      <parent link="${prefix}${fingerprefix}_inner_finger" />
+      <child link="${prefix}${fingerprefix}_pad_contact" />
+    </joint>
+  </xacro:macro>
   <xacro:macro name="onrobot_rg6" params="prefix">
     <xacro:onrobot_rg6_base_link prefix="${prefix}"/>
@@ -144,4 +160,8 @@
     <xacro:finger_joint prefix="${prefix}"/>
     <xacro:right_outer_knuckle_joint prefix="${prefix}"/>
+    <xacro:pad_contact prefix="${prefix}" fingerprefix="left"/>
+    <!-- <xacro:pad_contact prefix="${prefix}" fingerprefix="right"/> -->
+    <xacro:pad_contact_joint prefix="${prefix}" fingerprefix="left"/>
+    <!-- <xacro:pad_contact_joint prefix="${prefix}" fingerprefix="right"/> -->
     <xacro:onrobot_rg6_transmission prefix="${prefix}"/>
     <xacro:onrobot_rg6_gazebo prefix="${prefix}"/>
