Commit message: Update rg2 urdf

File: onrobot_rg_description/urdf/onrobot_rg2.xacro (robot description, xacro)
@@ -24,9 +24,8 @@
       </collision>
     </link>
-    <link name="world"/>
     <joint name="joint0" type="fixed">
-        <parent link="world"/>
+        <parent link="tool0"/>
         <child link="${prefix}onrobot_rg2_base_link"/>
-        <origin xyz= "0. 0. 0." rpy="0. 0. 0." />
+        <origin xyz="0 0 0" rpy="0 0 1.5708" />
     </joint>
     <gazebo reference="${prefix}onrobot_rg2_base_link">
